Commit message: Robot moving in gazebo

File: description/gazebo_control.xacro (robot description, xacro)
@@ -9,13 +9,30 @@
           <right_joint>right_wheel_joint</right_joint>
           <!-- kinematics -->
-          <wheel_separation>1.2</wheel_separation>
-          <wheel_radius>0.4</wheel_radius> <!-- computed from <wheel_diameter> in the original plugin-->
+          <wheel_separation>0.154</wheel_separation>
+          <wheel_radius>0.025</wheel_radius> <!-- computed from <wheel_diameter> in the original plugin-->
           <topic>cmd_vel</topic> <!-- from <commant_topic> -->
           <odom_publish_frequency>1</odom_publish_frequency>
-          <!-- <odom_topic>odometry</odom_topic>
+          <odom_topic>odometry</odom_topic>
           <frame_id>odom</frame_id>
           <child_frame_id>base_link</child_frame_id>
-          <odom_publisher_frequency>30</odom_publisher_frequency>
           <tf_topic>tf</tf_topic> Short topic name for tf output -->
+      </plugin>
+      <plugin
+        filename="gz-sim-odometry-publisher-system"
+        name="gz::sim::systems::OdometryPublisher">
+        <odom_frame>odom</odom_frame>
+        <robot_base_frame>base_link</robot_base_frame>
+      </plugin>
+      <plugin
+        filename="gz-sim-joint-state-publisher-system"
+        name="gz::sim::systems::JointStatePublisher">
+      </plugin>
+      <plugin
+        filename="gz-sim-pose-publisher-system"
+        name="gz::sim::systems::PosePublisher">
+        <publish_link_pose>true</publish_link_pose>
+        <use_pose_vector_msg>true</use_pose_vector_msg>
+        <static_publisher>true</static_publisher>
+        <static_update_frequency>1</static_update_frequency>
       </plugin>
   </gazebo>

File: description/robot.urdf.xacro (robot description, xacro)
@@ -4,4 +4,5 @@
     <xacro:include filename="robot_core.xacro"/>
     <xacro:include filename="gazebo_control.xacro"/>
+    <!--<xacro:include filename="lidar.xacro"/>-->
     <!-- <link name="base link"></link> -->
 </robot>

File: description/robot_core.xacro (robot description, xacro)
@@ -59,4 +59,17 @@
                 <cylinder radius="0.025" length="0.018"/>
             </geometry>
+            <surface>
+                <friction>
+                    <ode>
+                        <mu>100000.0</mu>
+                        <mu2>100000.0</mu2>
+                    </ode>
+                </friction>
+                <contact>
+                    <ode>
+                        <min_depth>0.003</min_depth>
+                    </ode>
+                </contact>
+            </surface>
         </collision>
         <xacro:inertial_cylinder mass="0.03" length="0.018" radius="0.025">
@@ -96,5 +109,5 @@
         <visual>
             <geometry>
-                <sphere radius="0.0114"/>
+                <sphere radius="0.025"/>
             </geometry>
             <material name="black"/>
@@ -102,10 +115,14 @@
         <collision>
             <geometry>
-                <sphere radius="0.0114"/>
+                <sphere radius="0.025"/>
             </geometry>
         </collision>
-        <xacro:inertial_sphere mass="0.036" radius="0.0114">
+        <xacro:inertial_sphere mass="0.02" radius="0.025">
             <origin xyz="0 0 0" rpy="0 0 0"/>
         </xacro:inertial_sphere>
     </link>
+    <gazebo reference="caster_wheel">
+        <mu1> 0 </mu1>
+        <mu2> 0 </mu2>
+    </gazebo>
 </robot>
