Commit message: Niedziałające sterowanie

File: description/robot.urdf.xacro (robot description, xacro)
@@ -1,9 +1,13 @@
 <?xml version="1.0"?>
 <robot xmlns:xacro="http://www.ros.org/wiki/xacro"  name="rumbek">
-    <!-- Example link -->
+    <xacro:arg name="use_ros2_control" default="true"/>
+    <xacro:if value="$(arg use_ros2_control)">
+        <xacro:include filename="ros2_control.xacro"/>
+    </xacro:if>
+    <xacro:unless value="$(arg use_ros2_control)">
+        <xacro:include filename="gazebo_control.xacro"/>
+    </xacro:unless>
     <xacro:include filename="robot_core.xacro"/>
-    <!-- <xacro:include filename="gazebo_control.xacro"/> -->
     <xacro:include filename="lidar.xacro"/>
-    <xacro:include filename="ros2_control.xacro"/>
     <!-- <link name="base link"></link> -->
 </robot>

File: description/ros2_control.xacro (robot description, xacro)
@@ -1,28 +1,64 @@
 <?xml version="1.0"?>
 <robot xmlns:xacro="http://www.ros.org/wiki/xacro">
-  <ros2_control name="GazeboSimSystem" type="system">
-    <hardware>
-      <plugin>gz_ros2_control/GazeboSimSystem</plugin>
-    </hardware>
-    <joint name="left_wheel_joint">
-      <command_interface name="velocity">
-        <param name="min">-10</param>
-        <param name="max">10</param>
-      </command_interface>
-      <state_interface name="velocity"/>
-      <state_interface name="position"/>
-    </joint>
-    <joint name="right_wheel_joint">
-      <command_interface name="velocity">
-        <param name="min">-10</param>
-        <param name="max">10</param>
-      </command_interface>
-      <state_interface name="velocity"/>
-      <state_interface name="position"/>
-    </joint>
-</ros2_control>
+  <!-- <xacro:unless value="$(arg sim_mode)"> -->
+    <xacro:macro name="diffbot_ros2_control" params="name prefix use_mock_hardware">
+      <ros2_control name="${name}" type="system">
+        <xacro:unless value="${use_mock_hardware}">
+          <hardware>
+            <plugin>diffdrive_pico/DiffBotSystemHardware</plugin>
+              <param name="left_wheel_name">left_wheel_joint</param>
+              <param name="right_wheel_name">right_wheel_joint</param>
+              <param name="device">/dev/ttyACM0</param>
+              <param name="baud_rate">115200</param>
+              <param name="timeout">10</param>
+              <param name="enc_counts_per_rev">1958</param>
+          </hardware>
+        </xacro:unless>
+        <xacro:if value="${use_mock_hardware}">
+          <hardware>
+            <plugin>mock_components/GenericSystem</plugin>
+            <param name="calculate_dynamics">true</param>
+          </hardware>
+        </xacro:if>
+        <joint name="${prefix}left_wheel_joint">
+          <command_interface name="velocity"/>
+          <state_interface name="position"/>
+          <state_interface name="velocity"/>
+        </joint>
+        <joint name="${prefix}right_wheel_joint">
+          <command_interface name="velocity"/>
+          <state_interface name="position"/>
+          <state_interface name="velocity"/>
+        </joint>
+      </ros2_control>
+    </xacro:macro>
+  <!-- </xacro:unless>
+  <xacro:if value="$(sim_mode)">
+    <ros2_control name="GazeboSimSystem" type="system">
+      <hardware>
+        <plugin>gz_ros2_control/GazeboSimSystem</plugin>
+      </hardware>
+      <joint name="left_wheel_joint">
+        <command_interface name="velocity">
+          <param name="min">-10</param>
+          <param name="max">10</param>
+        </command_interface>
+        <state_interface name="velocity"/>
+        <state_interface name="position"/>
+      </joint>
+      <joint name="right_wheel_joint">
+        <command_interface name="velocity">
+          <param name="min">-10</param>
+          <param name="max">10</param>
+        </command_interface>
+        <state_interface name="velocity"/>
+        <state_interface name="position"/>
+      </joint>
+    <ros2_control>
+  </xacro:if> -->
 <gazebo>
   <plugin filename="gz_ros2_control-system" name="gz_ros2_control::GazeboSimROS2ControlPlugin">
     <parameters>$(find my_bot)/config/my_controllers.yaml</parameters>
+    <parameters>$(find my_bot)/config/sim_control.yaml</parameters>
   </plugin>
 </gazebo>
