Commit message: działa sterowanie fizycznymi silnikami
ros2 launch my_bot launch_robot.launch.py
ros2 run teleop_twist_keyboard teleop_twist_keyboard --ros-args -r /cmd_vel:=/diff_cont/cmd_vel -p stamped:=true -p use_sim_time:=true

File: description/ros2_control.xacro (robot description, xacro)
@@ -2,35 +2,25 @@
 <robot xmlns:xacro="http://www.ros.org/wiki/xacro">
   <!-- <xacro:unless value="$(arg sim_mode)"> -->
-    <xacro:macro name="diffbot_ros2_control" params="name prefix use_mock_hardware">
-      <ros2_control name="${name}" type="system">
-        <xacro:unless value="${use_mock_hardware}">
-          <hardware>
-            <plugin>diffdrive_pico/DiffBotSystemHardware</plugin>
-              <param name="left_wheel_name">left_wheel_joint</param>
-              <param name="right_wheel_name">right_wheel_joint</param>
-              <param name="device">/dev/ttyACM0</param>
-              <param name="baud_rate">115200</param>
-              <param name="timeout">10</param>
-              <param name="enc_counts_per_rev">1958</param>
-          </hardware>
-        </xacro:unless>
-        <xacro:if value="${use_mock_hardware}">
-          <hardware>
-            <plugin>mock_components/GenericSystem</plugin>
-            <param name="calculate_dynamics">true</param>
-          </hardware>
-        </xacro:if>
-        <joint name="${prefix}left_wheel_joint">
-          <command_interface name="velocity"/>
-          <state_interface name="position"/>
-          <state_interface name="velocity"/>
-        </joint>
-        <joint name="${prefix}right_wheel_joint">
-          <command_interface name="velocity"/>
-          <state_interface name="position"/>
-          <state_interface name="velocity"/>
-        </joint>
-      </ros2_control>
-    </xacro:macro>
+  <ros2_control name="rumbek_control" type="system">
+    <hardware>
+      <plugin>diffdrive_pico/DiffBotSystemHardware</plugin>
+        <param name="left_wheel_name">left_wheel_joint</param>
+        <param name="right_wheel_name">right_wheel_joint</param>
+        <param name="device">/dev/ttyACM0</param>
+        <param name="baud_rate">115200</param>
+        <param name="timeout">10</param>
+        <param name="enc_counts_per_rev">1958</param>
+    </hardware>
+    <joint name="left_wheel_joint">
+      <command_interface name="velocity"/>
+      <state_interface name="position"/>
+      <state_interface name="velocity"/>
+    </joint>
+    <joint name="right_wheel_joint">
+      <command_interface name="velocity"/>
+      <state_interface name="position"/>
+      <state_interface name="velocity"/>
+    </joint>
+  </ros2_control>
   <!-- </xacro:unless>
   <xacro:if value="$(sim_mode)">
