Commit message: Created core URDF

File: description/robot_core.xacro (robot description, xacro)
@@ -1,4 +1,5 @@
 <?xml version="1.0"?>
 <robot xmlns:xacro="http://www.ros.org/wiki/xacro">
+    <xacro:include filename="inertial_macros.xacro"/>
     <material name="white">
         <color rgba=" 1 1 1 1" />
@@ -13,19 +14,98 @@
         <color rgba=" 0 0 0 1" />
     </material>
+    <!-- BASE LINK -->
     <link name="base_link">
     </link>
+    <!-- CHASSIS LINK-->
     <joint name ="chassis_joint" type="fixed">
         <parent link="base_link"/>
         <child link="chassis"/>
-        <origin xyz="-0.07 0 0"/>
+        <origin xyz="-0.1 0 0"/>
     </joint>
     <link name="chassis">
         <visual>
-            <origin xyz="0.08 0 0.04"/>
+            <origin xyz="0.16 0 0.04"/>
             <geometry>
-                <box size="0.16 0.16 0.08"/>
+                <box size="0.32 0.32 0.08"/>
             </geometry>
             <material name="white"/>
         </visual>
+        <collision>
+            <origin xyz="0.16 0 0.04"/>
+            <geometry>
+                <box size="0.32 0.32 0.08"/>
+            </geometry>
+        </collision>
+        <xacro:inertial_box mass="1" x="0.32" y="0.32" z="0.08">
+            <origin xyz="0.16 0 0.04" rpy="0 0 0 "/>
+        </xacro:inertial_box>
+    </link>
+    <!-- LEFT WHEEL LINK-->
+    <joint name='left_wheel_joint' type="continuous">
+        <parent link="base_link"/>
+        <child link="left_wheel"/>
+        <origin xyz="0 0.077 0 " rpy="-${pi/2} 0 0"/>
+        <axis xyz="0 0 1"/>
+    </joint>
+    <link name="left_wheel">
+        <visual>
+            <geometry>
+                <cylinder radius="0.025" length="0.018"/>
+            </geometry>
+            <material name="blue"/>
+        </visual>
+        <collision>
+            <geometry>
+                <cylinder radius="0.025" length="0.018"/>
+            </geometry>
+        </collision>
+        <xacro:inertial_cylinder mass="0.03" length="0.018" radius="0.025">
+            <origin xyz="0 0 0" rpy="0 0 0"/>
+        </xacro:inertial_cylinder>
+    </link>
+    <!-- RIGHT WHEEL LINK-->
+    <joint name='right_wheel_joint' type="continuous">
+        <parent link="base_link"/>
+        <child link="right_wheel"/>
+        <origin xyz="0 -0.077 0 " rpy="${pi/2} 0 0"/>
+        <axis xyz="0 0 -1"/>
+    </joint>
+    <link name="right_wheel">
+        <visual>
+            <geometry>
+                <cylinder radius="0.025" length="0.018"/>
+            </geometry>
+            <material name="blue"/>
+        </visual>
+        <collision>
+            <geometry>
+                <cylinder radius="0.025" length="0.018"/>
+            </geometry>
+        </collision>
+        <xacro:inertial_cylinder mass="0.03" length="0.018" radius="0.025">
+            <origin xyz="0 0 0" rpy="0 0 0"/>
+        </xacro:inertial_cylinder>
+    </link>
+    <!-- CASTER WHEEL LINK-->
+    <joint name="caster_wheel_joint" type="fixed">
+        <parent link="chassis"/>
+        <child link="caster_wheel"/>
+        <origin xyz="0.24 0 0 "/>
+    </joint>
+    <link name="caster_wheel">
+        <visual>
+            <geometry>
+                <sphere radius="0.0114"/>
+            </geometry>
+            <material name="black"/>
+        </visual>
+        <collision>
+            <geometry>
+                <sphere radius="0.0114"/>
+            </geometry>
+        </collision>
+        <xacro:inertial_sphere mass="0.036" radius="0.0114">
+            <origin xyz="0 0 0" rpy="0 0 0"/>
+        </xacro:inertial_sphere>
     </link>
 </robot>

Commit message: Slam added

File: description/robot_core.xacro (robot description, xacro)
@@ -16,4 +16,12 @@
     <!-- BASE LINK -->
     <link name="base_link">
+    </link>
+    <!-- BASE FOOTPRINT LINK-->
+    <joint name="base_footprint_joint" type="fixed">
+        <parent link="base_link"/>
+        <child link="base_footprint"/>
+        <origin xyz="0 0 0" rpy="0 0 0 "/>
+    </joint>
+    <link="base_footprint">
     </link>
     <!-- CHASSIS LINK-->
@@ -126,3 +134,25 @@
         <mu2> 0 </mu2>
     </gazebo>
+    <!-- LASER FRAME-->
+    <joint name="laser_frame_joint" type="fixed">
+        <parent link="base_link"/>
+        <child link="laser_frame"/>
+        <origin xyz="0 0 0" rpy="0 0 0"/>
+    </joint>
+    <link name="laser_frame">
+        <visual>
+            <geometry>
+                <cylinder radius="0.025" length="0.018"/>
+            </geometry>
+            <material name="orange"/>
+        </visual>
+        <collision>
+            <geometry>
+                <cylinder radius="0.025" length="0.018"/>
+            </geometry>
+        </collision>
+        <xacro:inertial_cylinder mass="0.03" length="0.018" radius="0.025">
+            <origin xyz="0 0 0" rpy="0 0 0"/>
+        </xacro:inertial_cylinder>
+    </link>
 </robot>

Commit message: Fixing base_footprint

File: description/robot_core.xacro (robot description, xacro)
@@ -23,5 +23,5 @@
         <origin xyz="0 0 0" rpy="0 0 0 "/>
     </joint>
-    <link="base_footprint">
+    <link name="base_footprint">
     </link>
     <!-- CHASSIS LINK-->
